Commit message: Removed robot instance within the world such that it does not prohibit spawning of the robot. Customized robot wheel colors.

File: src/my_robot/urdf/my_robot.xacro (robot description, xacro)
@@ -170,3 +170,9 @@
 		</visual>
 	</link>
+<gazebo reference="left_wheel">
+    <material>Gazebo/Yellow</material>
+  </gazebo>
+  <gazebo reference="right_wheel">
+    <material>Gazebo/Black</material>
+  </gazebo>
 </robot>
